File: HarpyFC.brd (EAGLE design)
At the start: 35 x 41 mm, 103 parts, among them IC1 ICM-20689, IC2 STM32F722RGT, Q1 MOSFET-PCHANNEL, T1 2N7002E, U1 MP2307, U2 TPS63001, U3 MX25L6406EM2I-12G, Y1 8MHz

Commit message: outing in progress ..
Parts:
- moved P$19 3.00 mm to (33.5, 12.5)
- moved P$2 3.00 mm to (33.5, 9.50)
- moved L1 2.12 mm to (20.5, 18.0)
- moved C9 1.85 mm to (12.9, 12.7), turned to 270 degrees
- moved P$1 1.50 mm to (26.5, 1.50)
- moved C11 1.42 mm to (28.9, 22.5)
- moved C10 1.41 mm to (18.6, 23.9), turned to 0 degrees
- moved P$24 1.40 mm to (27.9, 1.50)
- moved P$15 1.13 mm to (16.9, 23.4)
- moved C5 1.12 mm to (29.5, 19.8), turned to 270 degrees
- moved R16 1.01 mm to (20.6, 23.9), turned to 0 degrees
- moved Y1 0.95 mm to (25.2, 26.7)
- moved R8 0.82 mm to (9.27, 8.79), turned to 0 degrees
- moved C7 0.51 mm to (15.2, 12.2)
- moved P$14 0.51 mm to (14.3, 20.8)
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Routing:
- net GND: track 33.5 -> 213.2 mm, vias 0 -> 10
- net VDD: track 37.3 -> 103.9 mm, vias 0 -> 5
- net VCC: track 59.1 -> 113.4 mm, vias 0 -> 3
- net UART5_RX: track 0.00 -> 49.4 mm, vias 0 -> 3
- net PPM: track 0.00 -> 37.0 mm, vias 0 -> 1
- net CURR: track 0.00 -> 36.8 mm, vias 0 -> 2
- net CAM_SWITCH: track 0.00 -> 36.0 mm, vias 0 -> 1
- net INT: track 0.00 -> 35.7 mm, vias 0 -> 2
- net VBAT_OUT: track 74.8 -> 109.2 mm, vias 0 -> 1
- net N$35: track 0.00 -> 32.9 mm
- net UART1_RX: track 0.00 -> 32.4 mm
- net UART1_TX: track 0.00 -> 30.1 mm
- net N$38: track 0.00 -> 27.5 mm
- net UART4_RX: track 0.00 -> 26.5 mm, vias 0 -> 1
- net UART5_TX: track 0.00 -> 26.2 mm, vias 0 -> 1
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
Commit message: routing finished.
Parts:
- moved C26 2.47 mm to (16.7, 21.9), turned to 0 degrees
- moved R10 2.24 mm to (11.2, 5.59), turned to 270 degrees
- moved C9 2.17 mm to (14.7, 13.9), turned to 180 degrees
- moved P$15 1.08 mm to (15.9, 24.0), turned to 0 degrees
- moved R9 0.63 mm to (14.1, 13.2)
- moved C1 0.50 mm to (10.3, 25.4)
- moved C2 0.50 mm to (9.29, 25.4)
- moved C20 0.50 mm to (13.0, 6.40)
- moved R11 0.40 mm to (13.1, 5.21)
- moved T1 0.20 mm to (29.1, 26.5)
- moved R16 0.10 mm to (20.6, 23.8)
- moved C10 0.10 mm to (18.6, 23.8)
Routing:
- net VDD: track 103.9 -> 175.9 mm, vias 5 -> 12
- net CAM_SWITCH: track 36.0 -> 47.0 mm
- net VBAT_OUT: track 109.2 -> 116.0 mm
- net SPI3_MOSI: track 33.9 -> 39.0 mm
- net GND: track 213.2 -> 217.4 mm, vias 10 -> 21
- net N$37: track 1.91 -> 5.60 mm
- net N$30: track 2.90 -> 5.96 mm
- net N$9: track 3.94 -> 1.32 mm
- net UART2_TX: track 2.11 -> 3.97 mm
- net UART5_TX: track 26.2 -> 27.9 mm
- net UART5_RX: track 49.4 -> 50.8 mm
- net INT: track 35.7 -> 37.0 mm
- net UART1_TX: track 30.1 -> 31.4 mm
- net VOUT: track 25.6 -> 26.6 mm
- net CURR: track 36.8 -> 37.8 mm
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- added copper zone on layer 1, net GND
- added copper zone on layer 16, net GND

Commit message: Modification suite a test n1
Parts:
- removed R10, R12: (no value), HarpyFC_Library:0402-TIGHT
- removed R11: (no value), HarpyFC_Library:0402
- C13, C14, C18, C19, C3, C9: device HarpyFC_Library:0402-TIGHT -> HarpyFC_Library:0603
- C24: device HarpyFC_Library:0402-TIGHT -> HarpyFC_Library:0805
- C25: value 100uF -> 22uF; device HarpyFC_Library:0402-TIGHT -> HarpyFC_Library:0805
- LED0, LED1, LED2: device HarpyFC_Library:LED-0603 -> HarpyFC_Library:0805
- R2: value (none) -> 100k
- R3: value (none) -> 6.8k
- R4: value (none) -> 44.2k
- R5: value (none) -> 10k
- moved C24 3.14 mm to (10.1, 11.8), turned to 270 degrees
- moved C3 1.35 mm to (5.90, 21.2), turned to 270 degrees
- moved C19 1.32 mm to (5.29, 22.6)
- moved C9 0.95 mm to (13.8, 13.6)
- moved R15 0.81 mm to (27.5, 33.8)
- moved LED2 0.80 mm to (24.7, 33.8)
- moved C13 0.73 mm to (22.9, 31.4)
- moved C7 0.66 mm to (14.8, 11.6), turned to 90 degrees
- moved R9 0.61 mm to (14.2, 13.8)
- moved C25 0.54 mm to (12.6, 11.5)
- moved R14 0.40 mm to (27.6, 32.1)
- moved LED1 0.35 mm to (24.7, 32.1)
- moved C18 0.20 mm to (7.53, 16.8)
- moved C14 0.20 mm to (26.7, 16.4)
- moved R7 0.10 mm to (5.99, 15.8)
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Connections:
- removed net N$30: R10.2, U$1.17
- removed net N$31: R11.2, U$1.18
- removed net N$33: R12.2, U$1.12
- new net N$5: C21.2, R8.2
- net BUZZ: now also IC2.61; no longer IC2.2
- net GND: now also LED0.2; no longer C21.2, C22.2, LED0.C, R8.2
- net N$32: now also LED0.1; no longer LED0.A
- net N$34: now also LED1.1; no longer LED1.A
- net N$35: now also LED1.2; no longer LED1.C
- net N$36: now also LED2.1; no longer LED2.A
- net N$38: now also LED2.2; no longer LED2.C
- net VCC: no longer R10.1, R11.1, R12.1
- net VIN: no longer R8.1
Routing:
- net GND: track 217.4 -> 199.1 mm, vias 21 -> 23
- net VDD: track 175.9 -> 183.1 mm
- net N$30: track 5.96 -> 0.00 mm
- net VIN: track 29.5 -> 25.8 mm
- net N$27: track 1.96 -> 5.52 mm
- net N$29: track 3.08 -> 5.95 mm
- net N$31: track 2.35 -> 0.00 mm
- net N$4: track 2.09 -> 0.00 mm
- net N$3: track 2.03 -> 0.00 mm
- net N$33: track 1.68 -> 0.00 mm
- net N$23: track 9.18 -> 10.2 mm
- net VBAT_OUT: track 116.0 -> 117.0 mm
- net N$9: track 1.32 -> 2.00 mm
- net VOUT: track 26.6 -> 27.3 mm
- net SW: track 12.5 -> 11.9 mm
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
Commit message: last modification, but not implemented on brd
Parts:
- moved C20 0.20 mm to (12.8, 6.40)
Connections:
- removed net N$3: C21.1, U$1.21
- removed net N$5: C21.2, R8.2
- new net S$1: U$1.19, U$1.3
- new net S$3: C23.1
- net VCC: no longer U$1.19, U$1.3
- net VIN: no longer C23.1
Routing:
- net VCC: track 112.5 -> 82.8 mm
- net S$1: track 0.00 -> 24.5 mm
- net VIN: track 25.8 -> 24.6 mm
