File: HarpyFC.sch (EAGLE design)
At the start: 127 parts, among them IC1 ICM-20689, IC2 STM32F722RGT, Q1 MOSFET-PCHANNEL, T1 2N7002E, U1 MP2307, U2 TPS63001, U3 MX25L6406EM2I-12G, U4 SN74LVC1G04DBVR, Y1 8MHz

Commit message: Routing in process
Parts:
- removed P$10, P$11, P$8, P$9: (no value), HarpyFC_Library:SIGNAL_PAD
- removed U$12, U$13, U$14, U$15, U$16, U$18, U$19, U$20, U$22, U$23, U$24, U$25, U$26, U$27, U$28, U$29, U$30, U$31, U$34, U$35: (no value), HarpyFC_Library:POWER_PAD
- removed U4: SN74LVC1G04DBVR, HarpyFC_Library:SN74LVC1G045L
- added CN1: (no value), HarpyFC_Library:JST_8PINJSTSH8
- R1, R5: value 10k -> (none); device HarpyFC_Library:RESISTOR0402 -> HarpyFC_Library:RESISTOR
- R10: value 1k -> (none); device HarpyFC_Library:RESISTOR0402 -> HarpyFC_Library:RESISTOR; SPICEPREFIX (none) -> R
- R11: value 1k -> (none)
- R12: value 1k -> (none); device HarpyFC_Library:RESISTOR0402 -> HarpyFC_Library:RESISTOR
- R13: value 330R -> (none); device HarpyFC_Library:RESISTOR0402 -> HarpyFC_Library:RESISTOR
- R14, R15: value 220R -> (none); device HarpyFC_Library:RESISTOR0402 -> HarpyFC_Library:RESISTOR
- R16: value 100R -> (none); device HarpyFC_Library:RESISTOR0402 -> HarpyFC_Library:RESISTOR
- R2: value 100k -> (none); device HarpyFC_Library:RESISTOR0402 -> HarpyFC_Library:RESISTOR
- R3: value 6.8k -> (none); device HarpyFC_Library:RESISTOR0402 -> HarpyFC_Library:RESISTOR
- R4: value 44.2k -> (none); device HarpyFC_Library:RESISTOR0402 -> HarpyFC_Library:RESISTOR
- R6, R7: value 22R -> (none); device HarpyFC_Library:RESISTOR0402 -> HarpyFC_Library:RESISTOR
- R8, R9: value 75R -> (none); device HarpyFC_Library:RESISTOR0402 -> HarpyFC_Library:RESISTOR
Connections:
- removed net USART1_RX: IC2G$1.PB6, U4.Y
- new net CURR: CN1.1, IC2G$1.PC2
- new net VBAT_IN: U$2.IP+@1, U$2.IP+@2, U$3.P$1
- net GND: now also CN1.8; no longer IC2G$1.PB7, IC2G$1.PB8, IC2G$1.PC2, U$12.P$1, U$22.P$1, U$23.P$1, U$24.P$1, U$25.P$1, U$26.P$1, U$27.P$1, U$28.P$1, U$29.P$1, U$30.P$1, U$31.P$1, U4.GND
- net M1: now also CN1.6
- net M2: now also CN1.5
- net M3: now also CN1.4
- net M4: now also CN1.3
- net M5: no longer P$8.P$1
- net M6: no longer P$9.P$1
- net M7: no longer P$10.P$1
- net M8: no longer P$11.P$1
- net SBUS_INV: now also IC2G$1.PB7; no longer U4.A
- net UART5_RX: now also CN1.2
- net VBAT_OUT: now also C14.1, CN1.7, R2.1, U$2.IP-@3, U$2.IP-@4, U$4.P$1, U1.IN; no longer U$13.P$1, U$14.P$1, U$15.P$1, U$16.P$1, U$18.P$1, U$19.P$1, U$20.P$1
- net VDD: no longer U$34.P$1, U$35.P$1, U4.VCC
- net VIN: no longer C14.1, R2.1, U$2.IP+@1, U$2.IP+@2, U$2.IP-@3, U$2.IP-@4, U$3.P$1, U$4.P$1, U1.IN
Other:
- note removed: "SBUS inverted"

Commit message: Modification suite a test n1
Parts:
- removed R12: (no value), HarpyFC_Library:RESISTOR
- added C28, C29: 10uF, HarpyFC_Library:CAP-0603
- added C30: 22uF, HarpyFC_Library:CAP-0603
- added R17: 680k, HarpyFC_Library:RESISTOR
- C13, C14, C18, C19, C3, C9: device HarpyFC_Library:CAP-0402-TIGHT -> HarpyFC_Library:CAP-0603
- C24: device HarpyFC_Library:CAP-0402-TIGHT -> HarpyFC_Library:CAP-0805
- C25: value 100uF -> 22uF; device HarpyFC_Library:CAP-0402-TIGHT -> HarpyFC_Library:CAP-0805
- LED0, LED1, LED2: device HarpyFC_Library:LED0603 -> HarpyFC_Library:LED
- R10: value (none) -> 100; SPICEPREFIX R -> (none)
- R11: value (none) -> 100k; device HarpyFC_Library:RESISTOR0402 -> HarpyFC_Library:RESISTOR
- R13, R14, R15: value (none) -> 330
- R16: value (none) -> 100
- R2: value (none) -> 100k
- R3: value (none) -> 6.8k
- R4: value (none) -> 44.2k
- R5: value (none) -> 10k
- R6, R7: value (none) -> 22
- R8, R9: value (none) -> 75
Connections:
- removed net M5: IC2G$1.PC4
- removed net N$24: C21.1, U$1.AVDD
- removed net N$25: C22.1, U$1.PVDD
- removed net N$30: R10.2, U$1.~VSYNC
- removed net N$31: R11.2, U$1.~HSYNC
- removed net N$33: R12.2, U$1.LOS
- new net ADC_VBAT: IC2G$1.PC4, R11.1, R17.2
- new net N$3: R10.2, U2.EN, U2.PS/SYNC, U2.VINA
- net BUZZ: now also IC2G$1.PB8; no longer IC2G$1.PC13
- net GND: now also C28.2, C29.2, C30.2, R17.1, R8.1; no longer R8.2
- net VBAT_OUT: now also C29.1, R11.2
- net VCC: now also C21.1, C22.1, C27.2, C30.1, U$1.AVDD, U$1.PVDD, U$11.P$1, U$2.VCC, U$36.P$1, U$37.P$1, U$38.P$1, U$7.P$1, U$9.P$1; no longer R10.1, R11.1, R12.1, USB1.VCC
- net VCC-REG: now also R10.1; no longer U2.EN, U2.PS/SYNC, U2.VINA
- net VDD: now also C28.1; no longer C27.2, U$11.P$1, U$2.VCC, U$36.P$1, U$37.P$1, U$38.P$1, U$7.P$1, U$9.P$1
- net VIN: now also R8.2; no longer R8.1
Other:
- moved on the sheet: C13, C18, C21, C22, C23, Q1, R10, R8

Commit message: last modification, but not implemented on brd
Parts:
- removed C28, C29: 10uF, HarpyFC_Library:CAP-0603
- removed C30: 22uF, HarpyFC_Library:CAP-0603
- removed R10: 100, HarpyFC_Library:RESISTOR
- removed R11: 100k, HarpyFC_Library:RESISTOR
- removed R17: 680k, HarpyFC_Library:RESISTOR
Connections:
- net ADC_VBAT: no longer R11.1, R17.2
- net GND: no longer C28.2, C29.2, C30.2, R17.1
- net N$3: no longer R10.2
- net VBAT_OUT: no longer C29.1, R11.2
- net VCC: no longer C30.1
- net VCC-REG: no longer R10.1
- net VDD: no longer C28.1
Changed lines of the file:
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@@
 <part name="VCC6" library="alienflight" deviceset="VCC" device=""/>
 <part name="VCC7" library="alienflight" deviceset="VCC" device=""/>
-<part name="C28" library="HarpyFC_Library" deviceset="CAP" device="-0603" value="10uF"/>
-<part name="R10" library="HarpyFC_Library" deviceset="RESISTOR" device="" value="100"/>
-<part name="C29" library="HarpyFC_Library" deviceset="CAP" device="-0603" value="10uF"/>
-<part name="C30" library="HarpyFC_Library" deviceset="CAP" device="-0603" value="22uF"/>
-<part name="R11" library="HarpyFC_Library" deviceset="RESISTOR" device="" value="100k"/>
-<part name="R17" library="HarpyFC_Library" deviceset="RESISTOR" device="" value="680k"/>
 <part name="GND45" library="supply1" library_urn="urn:adsk.eagle:library:371" deviceset="GND" device=""/>
 <part name="P+3" library="supply1" library_urn="urn:adsk.eagle:library:371" deviceset="VCC" device=""/>
@@
 <attribute name="VALUE" x="148.336" y="128.016" size="1.778" layer="96" rot="R180"/>
 </instance>
-<instance part="C28" gate="G$1" x="231.14" y="114.3" smashed="yes">
-<attribute name="NAME" x="232.664" y="117.221" size="1.778" layer="95" font="vector"/>
-<attribute name="VALUE" x="232.664" y="112.141" size="1.778" layer="96" font="vector"/>
-</instance>
-<instance part="R10" gate="G$1" x="185.42" y="132.08" smashed="yes">
-<attribute name="NAME" x="185.42" y="128.524" size="1.778" layer="95" font="vector" align="bottom-center"/>
-<attribute name="VALUE" x="185.42" y="128.016" size="1.778" layer="96" font="vector" align="top-center"/>
-</instance>
-<instance part="C29" gate="G$1" x="165.1" y="50.8" smashed="yes">
-<attribute name="NAME" x="160.528" y="53.467" size="1.778" layer="95" font="vector"/>
-<attribute name="VALUE" x="160.274" y="48.895" size="1.778" layer="96" font="vector"/>
-</instance>
-<instance part="C30" gate="G$1" x="241.3" y="43.18" smashed="yes">
-<attribute name="NAME" x="244.348" y="43.688" size="1.778" layer="95" font="vector"/>
-<attribute name="VALUE" x="244.348" y="41.148" size="1.778" layer="96" font="vector"/>
-</instance>
 </instances>
 <busses>
@@
 <pinref part="GND13" gate="1" pin="GND"/>
 <wire x1="170.18" y1="48.26" x2="170.18" y2="45.72" width="0.1524" layer="91"/>
-<pinref part="C29" gate="G$1" pin="2"/>
 <wire x1="165.1" y1="48.26" x2="165.1" y2="45.72" width="0.1524" layer="91"/>
 <wire x1="165.1" y1="45.72" x2="170.18" y2="45.72" width="0.1524" layer="91"/>
@@
 <pinref part="C13" gate="G$1" pin="2"/>
 <wire x1="236.22" y1="35.56" x2="236.22" y2="38.1" width="0.1524" layer="91"/>
-<pinref part="C30" gate="G$1" pin="2"/>
 <wire x1="236.22" y1="38.1" x2="236.22" y2="40.64" width="0.1524" layer="91"/>
 <wire x1="241.3" y1="40.64" x2="241.3" y2="38.1" width="0.1524" layer="91"/>
@@
 <pinref part="GND20" gate="1" pin="GND"/>
 <wire x1="223.52" y1="111.76" x2="223.52" y2="109.22" width="0.1524" layer="91"/>
-<pinref part="C28" gate="G$1" pin="2"/>
 <wire x1="231.14" y1="111.76" x2="231.14" y2="109.22" width="0.1524" layer="91"/>
 <wire x1="231.14" y1="109.22" x2="223.52" y2="109.22" width="0.1524" layer="91"/>
@@
 <wire x1="223.52" y1="134.62" x2="223.52" y2="144.78" width="0.1524" layer="91"/>
 <pinref part="SUPPLY7" gate="VDD" pin="VDD"/>
-<pinref part="C28" gate="G$1" pin="1"/>
 <wire x1="231.14" y1="119.38" x2="231.14" y2="134.62" width="0.1524" layer="91"/>
 <wire x1="231.14" y1="134.62" x2="223.52" y2="134.62" width="0.1524" layer="91"/>
@@
 <pinref part="U1" gate="G$1" pin="EN"/>
 <wire x1="228.6" y1="55.88" x2="215.9" y2="55.88" width="0.1524" layer="91"/>
-</segment>
-</net>
-<net name="VIN" class="0">
-<segment>
-<pinref part="C23" gate="G$1" pin="1"/>
-<label x="156.718" y="119.126" size="1.778" layer="95" rot="R180"/>
-<pinref part="R8" gate="G$1" pin="2"/>
-<wire x1="149.86" y1="119.38" x2="149.86" y2="116.84" width="0.1524" layer="91"/>
-<wire x1="149.86" y1="116.84" x2="149.86" y2="114.3" width="0.1524" layer="91"/>
-<wire x1="149.86" y1="116.84" x2="157.48" y2="116.84" width="0.1524" layer="91"/>
-<junction x="149.86" y="116.84"/>
 </segment>
 </net>
@@
 <wire x1="236.22" y1="48.26" x2="236.22" y2="50.8" width="0.1524" layer="91"/>
 <junction x="236.22" y="50.8"/>
-<pinref part="C30" gate="G$1" pin="1"/>
 <wire x1="241.3" y1="48.26" x2="241.3" y2="50.8" width="0.1524" layer="91"/>
 <junction x="241.3" y="50.8"/>
@@
 <junction x="177.8" y="134.62"/>
 <pinref part="C18" gate="G$1" pin="1"/>
-<pinref part="R10" gate="G$1" pin="1"/>
 <wire x1="177.8" y1="132.08" x2="177.8" y2="119.38" width="0.1524" layer="91"/>
 <wire x1="180.34" y1="132.08" x2="177.8" y2="132.08" width="0.1524" layer="91"/>
@@
 <segment>
 <pinref part="U1" gate="G$1" pin="IN"/>
-<wire x1="162.56" y1="55.88" x2="165.1" y2="55.88" width="0.1524" layer="91"/>
 <pinref part="C14" gate="G$1" pin="1"/>
 <junction x="170.18" y="55.88"/>
-<wire x1="165.1" y1="55.88" x2="170.18" y2="55.88" width="0.1524" layer="91"/>
+<wire x1="162.56" y1="55.88" x2="170.18" y2="55.88" width="0.1524" layer="91"/>
 <wire x1="170.18" y1="55.88" x2="190.5" y2="55.88" width="0.1524" layer="91"/>
 <label x="162.56" y="55.88" size="1.778" layer="95" rot="R90"/>
-<pinref part="C29" gate="G$1" pin="1"/>
-<junction x="165.1" y="55.88"/>
 </segment>
 <segment>
@@
 <wire x1="228.6" y1="68.58" x2="228.6" y2="66.04" width="0.1524" layer="91"/>
 <label x="228.6" y="68.58" size="1.778" layer="95" rot="R90"/>
-</segment>
-</net>
-<net name="N$6" class="0">
-<segment>
-<junction x="149.86" y="116.84"/>
 </segment>
 </net>
@@
 <pinref part="U2" gate="G$1" pin="PS/SYNC"/>
 <wire x1="193.04" y1="127" x2="193.04" y2="129.54" width="0.1524" layer="91"/>
-<pinref part="R10" gate="G$1" pin="2"/>
+</segment>
+</net>
+<net name="VIN" class="0">
+<segment>
+<pinref part="C23" gate="G$1" pin="1"/>
+<pinref part="R8" gate="G$1" pin="2"/>
+<wire x1="149.86" y1="119.38" x2="149.86" y2="114.3" width="0.1524" layer="91"/>
+<label x="149.86" y="116.84" size="1.778" layer="95"/>
 </segment>
 </net>
@@
 <attribute name="VALUE" x="168.91" y="32.512" size="1.778" layer="96"/>
 </instance>
-<instance part="R11" gate="G$1" x="157.48" y="60.96" smashed="yes" rot="R90">
-<attribute name="NAME" x="152.146" y="63.246" size="1.778" layer="95" font="vector" rot="R180" align="bottom-center"/>
-<attribute name="VALUE" x="152.908" y="58.42" size="1.778" layer="96" font="vector" rot="R180" align="top-center"/>
-</instance>
-<instance part="R17" gate="G$1" x="157.48" y="45.72" smashed="yes" rot="R90">
-<attribute name="NAME" x="152.908" y="48.006" size="1.778" layer="95" font="vector" rot="R180" align="bottom-center"/>
-<attribute name="VALUE" x="153.67" y="43.434" size="1.778" layer="96" font="vector" rot="R180" align="top-center"/>
-</instance>
 <instance part="GND45" gate="1" x="157.48" y="35.56" smashed="yes">
 <attribute name="VALUE" x="154.94" y="33.02" size="1.778" layer="96"/>
@@
 <segment>
 <pinref part="GND45" gate="1" pin="GND"/>
-<pinref part="R17" gate="G$1" pin="1"/>
 <wire x1="157.48" y1="38.1" x2="157.48" y2="40.64" width="0.1524" layer="91"/>
 </segment>
@@
 </segment>
 <segment>
-<pinref part="R11" gate="G$1" pin="2"/>
 <wire x1="157.48" y1="66.04" x2="157.48" y2="68.58" width="0.1524" layer="91"/>
 <label x="157.48" y="68.58" size="1.778" layer="95"/>
@@
 </segment>
 <segment>
-<pinref part="R17" gate="G$1" pin="2"/>
-<pinref part="R11" gate="G$1" pin="1"/>
 <wire x1="157.48" y1="50.8" x2="157.48" y2="53.34" width="0.1524" layer="91"/>
 <wire x1="157.48" y1="53.34" x2="157.48" y2="55.88" width="0.1524" layer="91"/>
